File: PWR.kicad_sch (KiCad schematic)
At the start: 37 parts, among them U2 LT8610, U3 LT8610

Commit message: revision 1: I2C pullups, USB LDO, etc.
Parts:
- removed C1: 10n, symbol Device:C
- removed C16: 470n, symbol Device:C
- removed C2: 1u, symbol Device:C
- removed C3: 4p7, symbol Device:C
- removed C4, C7: 100n, symbol Device:C
- removed C5: 47u, symbol Device:C
- removed C6: 4.7u, symbol Device:C
- removed D1: 28v zener, symbol Device:D_Zener
- removed L1: SPM3012T-4R7M-LR, symbol Device:L
- removed LED2: Red, LED_SMD:LED_0805_2012Metric_Pad1.15x1.40mm_HandSolder, symbol Device:LED
- removed R17: R, symbol Device:R
- removed R3: 52k, symbol Device:R
- removed R4: 680k, symbol Device:R
- removed R5: 130k, symbol Device:R
- removed R6: 100k, symbol Device:R
- removed U2: LT8610, Package_SO:MSOP-16-1EP_3x4.039mm_P0.5mm_EP1.651x2.845mm_ThermalVias, symbol Regulator_Switching:LT8610
- added TVS: PTVS5V0Z1USK, Diode_SMD:Nexperia_DSN1608-2_1.6x0.8mm, symbol Diode:PTVS5V0Z1USK
Connections:
- net 24V: now also TVS.1 (K)
- net GND: now also TVS.2 (A)
Other:
- note removed: "5v"
- note removed: "??? NMOS to ensure power transferred only when power good"
- moved on the sheet: C10, C11, C12, C13, C14, C15, C8, C9, L2, LED1, R10, R12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
