File: PCB/esp32.kicad_sch (KiCad schematic)
At the start: 21 parts, among them SW1 SW_Push, U1 ESP32-S3-WROOM-2, U4 74HC595, U6 TCA9548APWR

Commit message: Fixed UART, cleaned schematic, improved LDO
Parts:
- added R19: 1k, Resistor_SMD:R_0603_1608Metric_Pad0.98x0.95mm_HandSolder, symbol Device:R
- C1, C_dec1, C_dec2, C_dec3, C_dec4: footprint (none) -> Capacitor_SMD:C_0201_0603Metric_Pad0.64x0.40mm_HandSolder
- R11, R17, R23, R24, R25, R26, R27, R28, R3, R4, R5, R6: footprint (none) -> Resistor_SMD:R_0603_1608Metric_Pad0.98x0.95mm_HandSolder
- SW1: value SW_Push -> boot; footprint (none) -> Button_Switch_SMD:SW_SPST_SKQG_WithStem
- U4: footprint (none) -> Package_SO:SOIC-16_3.9x9.9mm_P1.27mm
Connections:
- net SDA: now also R28.1; no longer R28.2
- net TX: now also R19.1
- net 3v3 renamed +3V3
- net +3V3: now also R28.2; no longer R26.1, R28.1, R4.2, U6.10 (SD3), U6.5 (SC0)
- net RX renamed UART
- net UART: now also R19.2
- new net encoder0_SC: R4.2, U6.5 (SC0)
- new net encoder3_SD: R26.1, U6.10 (SD3)
- no-connect marks 23 -> 20
Other:
- note removed: "use alt encoder"
- moved on the sheet: C_dec2, C_dec3, R11, R17, R23, R24, R25, R26, R28, R4, R5, R6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

Commit message: PCB layout v1.0
Parts:
- added R42: 10k, Resistor_SMD:R_0603_1608Metric_Pad0.98x0.95mm_HandSolder, symbol Device:R
- BOOT1: renamed from SW1; value boot -> B3SL-1002P; footprint Button_Switch_SMD:SW_SPST_SKQG_WithStem -> Button_Switch_SMD:SW_SPST_B3SL-1002P
- C1: footprint Capacitor_SMD:C_0201_0603Metric_Pad0.64x0.40mm_HandSolder -> Capacitor_SMD:C_0603_1608Metric_Pad1.08x0.95mm_HandSolder
- C16: renamed from C_dec4; footprint Capacitor_SMD:C_0201_0603Metric_Pad0.64x0.40mm_HandSolder -> Capacitor_SMD:C_0603_1608Metric_Pad1.08x0.95mm_HandSolder
- C5: renamed from C_dec1; footprint Capacitor_SMD:C_0201_0603Metric_Pad0.64x0.40mm_HandSolder -> Capacitor_SMD:C_0603_1608Metric_Pad1.08x0.95mm_HandSolder
- C6: renamed from C_dec2; footprint Capacitor_SMD:C_0201_0603Metric_Pad0.64x0.40mm_HandSolder -> Capacitor_SMD:C_0603_1608Metric_Pad1.08x0.95mm_HandSolder
- C7: renamed from C_dec3; footprint Capacitor_SMD:C_0201_0603Metric_Pad0.64x0.40mm_HandSolder -> Capacitor_SMD:C_0603_1608Metric_Pad1.08x0.95mm_HandSolder
- R3: value 1k -> 10k
- U4: value 74HC595 -> 74HC595D
Connections:
- net GND: now also R42.2; no longer U1.16 (IO46)
- net reset: now reaches C1.1, R3.2, U1.3 (EN)
- net IO13 renamed endswitch0
- net IO14 renamed endswitch1
- net IO15 renamed endswitch2
- net IO16 renamed endswitch3
- new net: R42.1, U1.16 (IO46)
Other:
- moved on the sheet: BOOT1, C1, C16, C5, R19, R27, R28, R3, U1
