File: PCB/tmc2209_driver.kicad_sch (KiCad schematic)
At the start: 2 parts

Commit message: Fixed UART, cleaned schematic, improved LDO
Parts:
- removed R19: 1k, symbol Device:R
Connections:
- net 3v3 renamed +3V3
- net RX renamed UART
Changed lines of the file:
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@@
 		)
-	)
-	(junction
-		(at 83.82 57.15)
-		(diameter 0)
-		(color 0 0 0 0)
 	)
 	(no_connect
@@
 	(wire
 		(pts
-			(xy 115.57 52.07) (xy 123.19 52.07)
-		)
-		(stroke
-			(width 0)
-			(type default)
-		)
-	)
-	(wire
-		(pts
-			(xy 76.2 52.07) (xy 74.93 52.07)
-		)
-		(stroke
-			(width 0)
-			(type default)
-		)
-	)
-	(wire
-		(pts
-			(xy 83.82 52.07) (xy 83.82 57.15)
-		)
-		(stroke
-			(width 0)
-			(type default)
-		)
-	)
-	(wire
-		(pts
-			(xy 74.93 57.15) (xy 83.82 57.15)
+			(xy 115.57 52.07) (xy 121.92 52.07)
+		)
+		(stroke
+			(width 0)
+			(type default)
+		)
+	)
+	(wire
+		(pts
+			(xy 88.9 57.15) (xy 92.71 57.15)
 		)
 		(stroke
@@
 	(wire
 		(pts
-			(xy 92.71 57.15) (xy 83.82 57.15)
-		)
-		(stroke
-			(width 0)
-			(type default)
-		)
-	)
-	(wire
-		(pts
 			(xy 118.11 54.61) (xy 115.57 54.61)
 		)
@@
 		)
 	)
-	(global_label "RX"
-		(shape output)
-		(at 74.93 57.15 180)
+	(global_label "UART"
+		(shape bidirectional)
+		(at 88.9 57.15 180)
 		(fields_autoplaced yes)
 		(effects
@@
 		)
 		(property "Intersheetrefs" "${INTERSHEET_REFS}"
-			(at 69.4653 57.15 0)
-			(effects
-				(font
-					(size 1.27 1.27)
-				)
-				(justify right)
-				(hide yes)
-			)
-		)
-	)
-	(global_label "TX"
-		(shape input)
-		(at 74.93 52.07 180)
-		(fields_autoplaced yes)
-		(effects
-			(font
-				(size 1.27 1.27)
-			)
-			(justify right)
-		)
-		(property "Intersheetrefs" "${INTERSHEET_REFS}"
-			(at 69.7677 52.07 0)
+			(at 80.1468 57.15 0)
 			(effects
 				(font
@@
 		)
 	)
-	(global_label "3v3"
-		(shape input)
-		(at 123.19 52.07 0)
-		(fields_autoplaced yes)
-		(effects
-			(font
-				(size 1.27 1.27)
-			)
-			(justify left)
-		)
-		(property "Intersheetrefs" "${INTERSHEET_REFS}"
-			(at 129.5618 52.07 0)
-			(effects
-				(font
-					(size 1.27 1.27)
-				)
-				(justify left)
-				(hide yes)
-			)
-		)
-	)
 	(hierarchical_label "B1"
 		(shape output)
@@
 			)
 			(justify left)
-		)
-	)
-	(symbol
-		(lib_id "Device:R")
-		(at 80.01 52.07 90)
-		(unit 1)
-		(exclude_from_sim no)
-		(in_bom yes)
-		(on_board yes)
-		(dnp no)
-		(fields_autoplaced yes)
-		(property "Reference" "R19"
-			(at 80.01 45.72 90)
-			(effects
-				(font
-					(size 1.27 1.27)
-				)
-			)
-		)
-		(property "Value" "1k"
-			(at 80.01 48.26 90)
-			(effects
-				(font
-					(size 1.27 1.27)
-				)
-			)
-		)
-		(property "Footprint" ""
-			(at 80.01 53.848 90)
-			(effects
-				(font
-					(size 1.27 1.27)
-				)
-				(hide yes)
-			)
-		)
-		(property "Datasheet" "~"
-			(at 80.01 52.07 0)
-			(effects
-				(font
-					(size 1.27 1.27)
-				)
-				(hide yes)
-			)
-		)
-		(property "Description" "Resistor"
-			(at 80.01 52.07 0)
-			(effects
-				(font
-					(size 1.27 1.27)
-				)
-				(hide yes)
-			)
-		)
-		(pin "2"
-		)
-		(pin "1"
-		)
-		(instances
-			(project ""
-				(path "/29a68080-a031-4f05-96b8-20ecd97fb7f6/437963f2-c308-4c55-baad-71afe821dfae"
-					(reference "R19")
-					(unit 1)
-				)
-				(path "/29a68080-a031-4f05-96b8-20ecd97fb7f6/4e92f28f-87aa-471e-b28c-960df080128b"
-					(reference "R22")
-					(unit 1)
-				)
-				(path "/29a68080-a031-4f05-96b8-20ecd97fb7f6/88318efe-951a-468c-99b4-5591dceb2a51"
-					(reference "R21")
-					(unit 1)
-				)
-				(path "/29a68080-a031-4f05-96b8-20ecd97fb7f6/dfef7ec9-15bf-4f96-a727-1112cdb742ee"
-					(reference "R20")
-					(unit 1)
-				)
-			)
 		)
 	)
@@
 					(unit 1)
 				)
+			)
+		)
+	)
+	(symbol
+		(lib_id "power:+3V3")
+		(at 121.92 52.07 270)
+		(unit 1)
+		(exclude_from_sim no)
+		(in_bom yes)
+		(on_board yes)
+		(dnp no)
+		(fields_autoplaced yes)
+		(property "Reference" "#PWR017"
+			(at 118.11 52.07 0)
+			(effects
+				(font
+					(size 1.27 1.27)
+				)
+				(hide yes)
+			)
+		)
+		(property "Value" "+3V3"
+			(at 125.73 52.0699 90)
+			(effects
+				(font
+					(size 1.27 1.27)
+				)
+				(justify left)
+			)
+		)
+		(property "Footprint" ""
+			(at 121.92 52.07 0)
+			(effects
+				(font
+					(size 1.27 1.27)
+				)
+				(hide yes)
+			)
+		)
+		(property "Datasheet" ""
+			(at 121.92 52.07 0)
+			(effects
+				(font
+					(size 1.27 1.27)
+				)
+				(hide yes)
+			)
+		)
+		(property "Description" "Power symbol creates a global label with name \"+3V3\""
+			(at 121.92 52.07 0)
+			(effects
+				(font
+					(size 1.27 1.27)
+				)
+				(hide yes)
+			)
+		)
+		(pin "1"
+		)
+		(instances
+			(project ""
+				(path "/29a68080-a031-4f05-96b8-20ecd97fb7f6/437963f2-c308-4c55-baad-71afe821dfae"
+					(reference "#PWR017")
+					(unit 1)
+				)
+				(path "/29a68080-a031-4f05-96b8-20ecd97fb7f6/4e92f28f-87aa-471e-b28c-960df080128b"
+					(reference "#PWR020")
+					(unit 1)
+				)
+				(path "/29a68080-a031-4f05-96b8-20ecd97fb7f6/88318efe-951a-468c-99b4-5591dceb2a51"
+					(reference "#PWR019")
+					(unit 1)
+				)
+				(path "/29a68080-a031-4f05-96b8-20ecd97fb7f6/dfef7ec9-15bf-4f96-a727-1112cdb742ee"
+					(reference "#PWR018")
+					(unit 1)
+				)

Commit message: PCB layout v1.0
Parts:
- removed BOB-0: ~, symbol VNLib:TMC2209-LA_BOB
- added BOB-0: ~, VNfootprints:TMC2209_SilentStepStick, symbol VNLib:TMC2209-silentstepstick
- added C17: 4u7, Capacitor_SMD:C_0805_2012Metric_Pad1.18x1.45mm_HandSolder, symbol Device:C
- added C21: 1u, Capacitor_SMD:C_0603_1608Metric_Pad1.08x0.95mm_HandSolder, symbol Device:C
Connections:
- net +3V3: now also BOB-0.4 (VIO), C21.2
- net A1: now also BOB-0.8 (M1A)
- net A2: now also BOB-0.10 (M2A)
- net B1: now also BOB-0.6 (M1B)
- net B2: now also BOB-0.12 (M2B)
- net DIR: now also BOB-0.1 (DIR)
- net EN: now also BOB-0.15 (EN)
- net GND: now also BOB-0.14 (GND), BOB-0.2 (GND), C17.2, C21.1
- net MS1: now also BOB-0.13 (MS1)
- net MS2: now also BOB-0.11 (MS2)
- net STEP: now also BOB-0.3 (STEP)
- net UART: now also BOB-0.7 (UART)
- new net 24V: BOB-0.16 (+VM), C17.1

Commit message: pcb version ready for final check
Parts:
- added C25: 100uF/50V, Capacitor_SMD:CP_Elec_8x10.5, symbol Device:C_Polarized
- BOB-0: value ~ -> (none)
Connections:
- net 24V: now also C25.1
- net GND: now also C25.2
Other:
- note removed: "potentially diode OR the diagnostic together to interrupt esp to check faulty friver via uart cost: 1 GPIO"

Commit message: [pcb] Final processing and export of production data
Parts:
- removed C17: 4u7, Capacitor_SMD:C_0805_2012Metric_Pad1.18x1.45mm_HandSolder, symbol Device:C
- added F1: Fuse, Fuse:Fuse_1812_4532Metric_Pad1.30x3.40mm_HandSolder, symbol Device:Fuse
Connections:
- net 24V: no longer names the net of BOB-0.16 (+VM), C25.1
- net 24V: now also F1.2
- new net MOT_POWER: F1.1
Changed lines of the file:
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@@
-	)
-	(junction
-		(at 118.11 67.31)
-		(diameter 0)
-		(color 0 0 0 0)
 	)
 	(junction
@@
 	)
 	(junction
-		(at 125.73 67.31)
-		(diameter 0)
-		(color 0 0 0 0)
-	)
-	(junction
 		(at 125.73 73.66)
 		(diameter 0)
@@
 	(wire
 		(pts
-			(xy 125.73 73.66) (xy 125.73 67.31)
+			(xy 125.73 64.77) (xy 125.73 73.66)
 		)
 		(stroke
@@
 	(wire
 		(pts
-			(xy 125.73 64.77) (xy 125.73 67.31)
-		)
-		(stroke
-			(width 0)
-			(type default)
-		)
-	)
-	(wire
-		(pts
 			(xy 125.73 74.93) (xy 125.73 73.66)
 		)
@@
 	(wire
 		(pts
+			(xy 116.84 86.36) (xy 118.11 86.36)
+		)
+		(stroke
+			(width 0)
+			(type default)
+		)
+	)
+	(wire
+		(pts
 			(xy 115.57 62.23) (xy 118.11 62.23)
 		)
@@
 	(wire
 		(pts
+			(xy 102.87 86.36) (xy 109.22 86.36)
+		)
+		(stroke
+			(width 0)
+			(type default)
+		)
+	)
+	(wire
+		(pts
+			(xy 118.11 73.66) (xy 118.11 86.36)
+		)
+		(stroke
+			(width 0)
+			(type default)
+		)
+	)
+	(wire
+		(pts
 			(xy 91.44 62.23) (xy 92.71 62.23)
 		)
@@
 		(pts
 			(xy 91.44 67.31) (xy 92.71 67.31)
-		)
-		(stroke
-			(width 0)
-			(type default)
-		)
-	)
-	(wire
-		(pts
-			(xy 118.11 73.66) (xy 118.11 76.2)
 		)
 		(stroke
@@
 		)
 	)
-	(global_label "24V"
-		(shape input)
-		(at 118.11 76.2 270)
-		(fields_autoplaced yes)
-		(effects
-			(font
-				(size 1.27 1.27)
-			)
-			(justify right)
-		)
-		(property "Intersheetrefs" "${INTERSHEET_REFS}"
-			(at 118.11 82.6928 90)
-			(hide yes)
-			(show_name no)
-			(do_not_autoplace no)
-			(effects
-				(font
-					(size 1.27 1.27)
-				)
-				(justify right)
-			)
-		)
-	)
 	(hierarchical_label "B1"
 		(shape output)
@@
 			)
 			(justify left)
+		)
+	)
+	(hierarchical_label "MOT_POWER"
+		(shape input)
+		(at 102.87 86.36 180)
+		(effects
+			(font
+				(size 1.27 1.27)
+			)
+			(justify right)
 		)
 	)
@@
 	)
 	(symbol
+		(lib_id "Device:Fuse")
+		(at 113.03 86.36 90)
+		(unit 1)
+		(body_style 1)
+		(exclude_from_sim no)
+		(in_bom yes)
+		(on_board yes)
+		(in_pos_files yes)
+		(dnp no)
+		(fields_autoplaced yes)
+		(property "Reference" "F1"
+			(at 113.03 80.01 90)
+			(show_name no)
+			(do_not_autoplace no)
+			(effects
+				(font
+					(size 1.27 1.27)
+				)
+			)
+		)
+		(property "Value" "Fuse"
+			(at 113.03 82.55 90)
+			(show_name no)
+			(do_not_autoplace no)
+			(effects
+				(font
+					(size 1.27 1.27)
+				)
+			)
+		)
+		(property "Footprint" "Fuse:Fuse_1812_4532Metric_Pad1.30x3.40mm_HandSolder"
+			(at 113.03 88.138 90)
+			(hide yes)
+			(show_name no)
+			(do_not_autoplace no)
+			(effects
+				(font
+					(size 1.27 1.27)
+				)
+			)
+		)
+		(property "Datasheet" ""
+			(at 113.03 86.36 0)
+			(hide yes)
+			(show_name no)
+			(do_not_autoplace no)
+			(effects
+				(font
+					(size 1.27 1.27)
+				)
+			)
+		)
+		(property "Description" "Fuse"
+			(at 113.03 86.36 0)
+			(hide yes)
+			(show_name no)
+			(do_not_autoplace no)
+			(effects
+				(font
+					(size 1.27 1.27)
+				)
+			)
+		)
+		(pin "2"
+		)
+		(pin "1"
+		)
+		(instances
+			(project "esp32stepper"
+				(path "/29a68080-a031-4f05-96b8-20ecd97fb7f6/437963f2-c308-4c55-baad-71afe821dfae"
+					(reference "F1")
+					(unit 1)
+				)
+				(path "/29a68080-a031-4f05-96b8-20ecd97fb7f6/4e92f28f-87aa-471e-b28c-960df080128b"
+					(reference "F5")
+					(unit 1)
+				)
+				(path "/29a68080-a031-4f05-96b8-20ecd97fb7f6/88318efe-951a-468c-99b4-5591dceb2a51"
+					(reference "F4")
+					(unit 1)
+				)
+				(path "/29a68080-a031-4f05-96b8-20ecd97fb7f6/dfef7ec9-15bf-4f96-a727-1112cdb742ee"
+					(reference "F3")
+					(unit 1)
+				)
+			)
+		)
+	)
+	(symbol
 		(lib_id "Device:C_Polarized")
 		(at 121.92 73.66 90)
@@
 					(unit 1)
 				)
-			)
-		)
-	)
-	(symbol
-		(lib_id "Device:C")
-		(at 121.92 67.31 90)
-		(unit 1)
-		(body_style 1)
-		(exclude_from_sim no)
-		(in_bom yes)
-		(on_board yes)
-		(in_pos_files yes)
-		(dnp no)
-		(property "Reference" "C17"
-			(at 119.126 66.04 90)
-			(show_name no)
-			(do_not_autoplace no)
-			(effects
-				(font
-					(size 1.27 1.27)
-				)
-			)
-		)
-		(property "Value" "4u7"
-			(at 124.714 68.834 90)
-			(show_name no)
-			(do_not_autoplace no)
-			(effects
-				(font
-					(size 1.27 1.27)
-				)
-			)
-		)
-		(property "Footprint" "Capacitor_SMD:C_0805_2012Metric_Pad1.18x1.45mm_HandSolder"
-			(at 125.73 66.3448 0)
-			(hide yes)
-			(show_name no)
-			(do_not_autoplace no)
-			(effects
-				(font
-					(size 1.27 1.27)
-				)
-			)
-		)
-		(property "Datasheet" ""
-			(at 121.92 67.31 0)
-			(hide yes)
-			(show_name no)
-			(do_not_autoplace no)
-			(effects
-				(font
-					(size 1.27 1.27)
-				)
-			)
-		)
-		(property "Description" "Unpolarized capacitor"
-			(at 121.92 67.31 0)
-			(hide yes)
-			(show_name no)
-			(do_not_autoplace no)
-			(effects
-				(font
-					(size 1.27 1.27)
-				)
-			)
-		)
-		(pin "1"
-		)
-		(pin "2"
-		)
-		(instances
-			(project "esp32stepper"
-				(path "/29a68080-a031-4f05-96b8-20ecd97fb7f6/437963f2-c308-4c55-baad-71afe821dfae"
-					(reference "C17")
-					(unit 1)
-				)
-				(path "/29a68080-a031-4f05-96b8-20ecd97fb7f6/4e92f28f-87aa-471e-b28c-960df080128b"
-					(reference "C20")
-					(unit 1)
-				)
-				(path "/29a68080-a031-4f05-96b8-20ecd97fb7f6/88318efe-951a-468c-99b4-5591dceb2a51"
-					(reference "C19")
-					(unit 1)
-				)
-				(path "/29a68080-a031-4f05-96b8-20ecd97fb7f6/dfef7ec9-15bf-4f96-a727-1112cdb742ee"
-					(reference "C18")
-					(unit 1)
-				)
